File: _devices/zeropc/diagram/KiCAD/ZeroPC.kicad_pcb (KiCad board)
At the start: 2 copper layers, 150 x 100 mm, 65 parts, among them IC1 Raspberry_Zero_2W, J1 EXT, J2 AudioJack, SW1 Esc, SW10 9, SW11 0, SW12 Dot, SW13 BS, SW14 Alt, SW15 Q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

Commit message: init
Parts:
- added C5: 100u, Capacitor_THT:CP_Radial_D5.0mm_P2.50mm, F.Cu at (129.5, 23.1)
- moved C2 1.40 mm to (129.5, 31.4)
Routing:
- net /3V3: track 161.2 -> 170.0 mm
- net /GND: track 373.9 -> 380.0 mm
- net Net-(C2-Pad2): track 19.0 -> 20.3 mm
