File: _devices/zeropc/diagram/KiCAD/ZeroPC.kicad_sch (KiCad schematic)
At the start: 60 parts, among them IC1 Raspberry_Zero_2W, J1 EXT, J2 AudioJack, SW1 Esc, SW10 9, SW11 0, SW12 Dot, SW13 BS, SW14 Alt, SW15 Q, SW16 W, SW17 E, SW18 R, SW19 T, SW2 1, SW20 Y, SW21 U, SW22 I, SW23 O, SW24 P, SW25 Tab, SW26 Shift, SW27 A, SW28 S, SW29 D, SW3 2, SW30 F, SW31 G, SW32 H, SW33 J, SW34 K, SW35 L, SW36 Up, SW37 Enter, SW38 Ctrl, SW39 Space, SW4 3, SW40 Z, SW41 X, SW42 C, SW43 V, SW44 B, SW45 N, SW46 M, SW47 Left, SW48 Down, SW49 Right, SW5 4, SW6 5, SW7 6, SW8 7, SW9 8

Commit message: init
Parts:
- added C5: 100u, Capacitor_THT:CP_Radial_D5.0mm_P2.50mm, symbol Device:C_Polarized
Connections:
- net 3V3: now also C5.1
- net GND: now also C5.2
Changed lines of the file:
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@@
 	(wire
 		(pts
+			(xy 220.98 76.2) (xy 220.98 81.28)
+		)
+		(stroke
+			(width 0)
+			(type default)
+		)
+	)
+	(wire
+		(pts
 			(xy 58.42 154.94) (xy 248.92 154.94)
 		)
@@
 	(wire
 		(pts
+			(xy 220.98 63.5) (xy 220.98 68.58)
+		)
+		(stroke
+			(width 0)
+			(type default)
+		)
+	)
+	(wire
+		(pts
 			(xy 104.14 147.32) (xy 104.14 152.4)
 		)
@@
 		)
 	)
+	(label "3V3"
+		(at 220.98 63.5 0)
+		(effects
+			(font
+				(size 1.27 1.27)
+			)
+			(justify left bottom)
+		)
+	)
 	(label "COL3"
 		(at 154.305 121.92 0)
@@
 		)
 	)
+	(label "GND"
+		(at 220.98 81.28 0)
+		(effects
+			(font
+				(size 1.27 1.27)
+			)
+			(justify left bottom)
+		)
+	)
 	(label "ROW0"
 		(at 177.8 157.48 0)
@@
 					(unit 1)
 				)
+			)
+		)
+	)
+	(symbol
+		(lib_id "Device:C_Polarized")
+		(at 220.98 72.39 0)
+		(unit 1)
+		(exclude_from_sim no)
+		(in_bom yes)
+		(on_board yes)
+		(dnp no)
+		(property "Reference" "C5"
+			(at 216.535 72.39 90)
+			(effects
+				(font
+					(size 1.27 1.27)
+				)
+			)
+		)
+		(property "Value" "100u"
+			(at 214.63 72.39 90)
+			(effects
+				(font
+					(size 1.27 1.27)
+				)
+			)
+		)
+		(property "Footprint" "Capacitor_THT:CP_Radial_D5.0mm_P2.50mm"
+			(at 221.9452 76.2 0)
+			(effects
+				(font
+					(size 1.27 1.27)
+				)
+				(hide yes)
+			)
+		)
+		(property "Datasheet" "~"
+			(at 220.98 72.39 0)
+			(effects
+				(font
+					(size 1.27 1.27)
+				)
+				(hide yes)
+			)
+		)
+		(property "Description" "Polarized capacitor"
+			(at 220.98 72.39 0)
+			(effects
+				(font
+					(size 1.27 1.27)
+				)
+				(hide yes)
+			)
+		)
+		(pin "2"
+		)
+		(pin "1"
+		)
+		(instances
+			(project "ZeroPC"
+				(path "/b3c66170-a1e8-49f2-a3c7-446e9ba3066c"
+					(reference "C5")
+					(unit 1)
+				)

Commit message: init
Other:
- note added: "SPI1_MOSI"
